File: TinyKey/KiCad/TinyKey.kicad_pcb (KiCad board)
At the start: 2 copper layers, 261.6 x 83.8 mm, 110 parts, among them SW0:0 ESC, SW0:1 Q, SW0:10 P, SW0:11 EQ, SW0:12 BACK_SP, SW0:2 W, SW0:3 E, SW0:4 R, SW0:5 T, SW0:6 Y, SW0:7 U, SW0:8 I, SW0:9 O, SW1:0 TAB, SW1:1 A, SW1:10 COL, SW1:11 ENTER, SW1:2 S, SW1:3 D, SW1:4 F, SW1:5 G, SW1:6 H, SW1:7 J, SW1:8 K, SW1:9 L, SW2:0 L_SHIFT, SW2:1 Z, SW2:10 UP, SW2:11 R_SHIFT, SW2:12 HOME, SW2:2 X, SW2:3 C, SW2:4 V, SW2:5 B, SW2:6 N, SW2:7 M, SW2:8 L_ANG, SW2:9 R_ANG, SW3:0 L_CTRL, SW3:1 WIN_MOD, SW3:10 DOWN, SW3:11 RIGHT, SW3:12 END, SW3:2 L_ALT, SW3:3 L_META, SW3:5 SPACE, SW3:8 FN_HYPER, SW3:9 LEFT

Commit message: BlackRose V1 complete, Updated TinyKey to V2
Parts:
- removed LED_GND: LED_GND, Pin_Headers:Pin_Header_Straight_1x01
- added C0-4: COL_0-4, Pin_Headers:Pin_Header_Straight_1x05, F.Cu at (72.0, 53.0)
- added C5-7: COL_5-7, Pin_Headers:Pin_Header_Straight_1x03, F.Cu at (88.0, 53.0)
- added C8-12: COL_8-13, Pin_Headers:Pin_Header_Straight_1x05, F.Cu at (207.0, 52.0)
- added G1: GND_OUT, Pin_Headers:Pin_Header_Straight_1x01, F.Cu at (213.0, 52.0)
- added LA1: LA, Pin_Headers:Pin_Header_Straight_1x01, F.Cu at (223.0, 52.0)
- added LB1: LB, Pin_Headers:Pin_Header_Straight_1x01, F.Cu at (220.0, 52.0)
- added LC1: LC, Pin_Headers:Pin_Header_Straight_1x01, F.Cu at (217.0, 52.0)
- added R0-3: ROW_0-3, Pin_Headers:Pin_Header_Straight_1x04, F.Cu at (21.0, 106.0)
- moved D3 30.7 mm to (45.0, 105.0)
- moved D47 25.9 mm to (273.2, 102.4)
- moved D48 25.9 mm to (270.0, 102.4)
- moved SW2:12 25.6 mm to (269.1, 116.7)
- moved L3 25.3 mm to (264.6, 51.7)
- moved R1 25.3 mm to (231.6, 53.0)
- moved R2 25.3 mm to (245.5, 53.0)
- moved R3 25.3 mm to (259.5, 53.0)
- moved L1 25.3 mm to (236.6, 51.7)
- moved L2 25.3 mm to (250.6, 51.7)
- moved D23 25.0 mm to (126.2, 126.2)
- moved D42 25.0 mm to (229.1, 61.4)
- moved D46 24.9 mm to (251.3, 61.6)
- moved SW2:0 24.6 mm to (35.7, 102.4)
- moved SW0:12 24.6 mm to (261.9, 64.3)
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Connections:
- R1 pad 1: /LED_A -> Net-(LA1-Pad1)
- R2 pad 1: /LED_B -> Net-(LB1-Pad1)
- R3 pad 1: /LED_C -> Net-(LC1-Pad1)
Routing:
- net /COL0: track 51.2 -> 146.1 mm
- net /ROW0: track 233.7 -> 317.9 mm
- net /COL7: track 43.9 -> 116.4 mm
- net /COL6: track 43.9 -> 100.8 mm
- net /COL12: track 56.9 -> 100.2 mm
- net Net-(LC1-Pad1): track 0.00 -> 40.2 mm
- net /COL1: track 68.7 -> 107.5 mm
- net /COL8: track 54.9 -> 93.1 mm
- net GND: track 38.1 -> 0.00 mm
- net /COL5: track 71.0 -> 107.3 mm
- net /COL11: track 56.8 -> 88.9 mm
- net /COL4: track 43.9 -> 73.8 mm
- net /ROW1: track 226.1 -> 252.7 mm
- net /COL9: track 52.8 -> 76.9 mm
- net Net-(LB1-Pad1): track 0.00 -> 23.1 mm
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Other:
- board size 261.6 x 83.8 mm -> 261 x 87 mm
- board text added: "KRYBOARD v2.0"
- board text added: "Z&P"
- board text removed: "KRYBOARD v1.0"
